Commit message: Update f1tenth_description.xacro

File: urdf/f1tenth_description.xacro (robot description, xacro)
@@ -44,5 +44,5 @@
     <origin xyz="0.46 -0.135 -0.180" rpy="1.57 0 3.14" />
     <geometry>
-      <mesh filename="package://f1tenth_urdf/urdf/meshes/chassis.stl" scale="0.000990 0.0009375 0.0009375"/>
+      <mesh filename="package://f1tenth_hardware_interface/urdf/meshes/chassis.stl" scale="0.000990 0.0009375 0.0009375"/>
     </geometry>
   </xacro:macro>
@@ -50,5 +50,5 @@
     <origin xyz="0 0 0" rpy="0 0 0" />
     <geometry>
-      <mesh filename="package://f1tenth_urdf/urdf/meshes/left_wheel.stl" />
+      <mesh filename="package://f1tenth_hardware_interface/urdf/meshes/left_wheel.stl" />
     </geometry>
   </xacro:macro>
@@ -56,5 +56,5 @@
     <origin xyz="0 0 0" rpy="0 0 0" />
     <geometry>
-      <mesh filename="package://f1tenth_urdf/urdf/meshes/right_wheel.stl" />
+      <mesh filename="package://f1tenth_hardware_interface/urdf/meshes/right_wheel.stl" />
     </geometry>
   </xacro:macro>
@@ -62,5 +62,5 @@
     <origin xyz="0 0 0" rpy="0 0 0" />
     <geometry>
-      <mesh filename="package://f1tenth_urdf/urdf/meshes/left_wheel.stl" />
+      <mesh filename="package://f1tenth_hardware_interface/urdf/meshes/left_wheel.stl" />
     </geometry>
   </xacro:macro>
@@ -68,5 +68,5 @@
     <origin xyz="0 0 0" rpy="0 0 0" />
     <geometry>
-      <mesh filename="package://f1tenth_urdf/urdf/meshes/right_wheel.stl" />
+      <mesh filename="package://f1tenth_hardware_interface/urdf/meshes/right_wheel.stl" />
     </geometry>
   </xacro:macro>
@@ -74,5 +74,5 @@
     <origin xyz="0 0 0" rpy="0 0 0" />
     <geometry>
-      <mesh filename="package://f1tenth_urdf/urdf/meshes/hinge.stl" />
+      <mesh filename="package://f1tenth_hardware_interface/urdf/meshes/hinge.stl" />
     </geometry>
   </xacro:macro>
@@ -80,5 +80,5 @@
     <origin xyz="0 0 0" rpy="0 0 0" />
     <geometry>
-      <mesh filename="package://f1tenth_urdf/urdf/meshes/hinge.stl" />
+      <mesh filename="package://f1tenth_hardware_interface/urdf/meshes/hinge.stl" />
     </geometry>
   </xacro:macro>
